Commit message: update

File: LGDXRobot2.urdf (robot description, URDF)
Before this commit: robot /Users/sam/Develop/lgdxrobot2-webots/LGDXRobot2.urdf, 19 links, 18 joints
Links:
- removed link BASE_CENTRE_SOLID
- removed link BASE_FRONT_SOLID
- removed link BASE_REAR_SOLID
- removed link BASE_TOP_SOLID
- added link solid_0
- added link solid_1
- added link solid_10
- added link solid_2
- added link solid_3
- added link solid_4
- added link solid_5
- added link solid_6
- added link solid_7
- added link solid_8
- added link solid_9
Joints:
- removed joint base_link_BASE_CENTRE_SOLID_joint
- removed joint base_link_BASE_FRONT_SOLID_joint
- removed joint base_link_BASE_REAR_SOLID_joint
- removed joint base_link_BASE_TOP_SOLID_joint
- added joint base_link_solid_0_joint: type fixed, parent base_link, child solid_0, origin xyz=-0.102 0 0.057 rpy=0 0 0
- added joint base_link_solid_1_joint: type fixed, parent base_link, child solid_1, origin xyz=0.138 0.0685 0.094 rpy=0 0 0
- added joint base_link_solid_2_joint: type fixed, parent base_link, child solid_2, origin xyz=0.138 -0.0685 0.094 rpy=0 0 0
- added joint base_link_solid_3_joint: type fixed, parent base_link, child solid_3, origin xyz=0.066 0.0685 0.094 rpy=0 0 0
- added joint base_link_solid_4_joint: type fixed, parent base_link, child solid_4, origin xyz=0.066 -0.0685 0.094 rpy=0 0 0
- added joint base_link_solid_5_joint: type fixed, parent base_link, child solid_5, origin xyz=-0.066 0.0685 0.094 rpy=0 0 0
- added joint base_link_solid_6_joint: type fixed, parent base_link, child solid_6, origin xyz=-0.066 -0.0685 0.094 rpy=0 0 0
- added joint base_link_solid_7_joint: type fixed, parent base_link, child solid_7, origin xyz=-0.138 0.0685 0.094 rpy=0 0 0
- added joint base_link_solid_8_joint: type fixed, parent base_link, child solid_8, origin xyz=-0.138 -0.0685 0.094 rpy=0 0 0
- added joint base_link_solid_9_joint: type fixed, parent base_link, child solid_9, origin xyz=0 0 0.129 rpy=0 0 0
- added joint base_link_solid_joint: type fixed, parent base_link, child solid, origin xyz=0.102 0 0.057 rpy=0 0 0
- joint base_link_camera_joint: origin xyz=0.1 0.01 -0.03 rpy=0 0 0 -> xyz=0.1 0.01 0.059 rpy=0 0 0
- joint base_link_lidar_joint: origin xyz=0 0 0.067 rpy=0 0 0 -> xyz=0 0 0.157 rpy=0 0 3.14159
- joint lidar_secondary_motor: child solid -> solid_10
- joint wheel1: origin xyz=0.1055 0.10251 -0.0545 rpy=1.5708 0 0 -> xyz=0.1055 0.1025 0.0375 rpy=1.5708 0 0
- joint wheel2: origin xyz=0.1055 -0.10249 -0.0545 rpy=1.5708 0 0 -> xyz=0.1055 -0.1025 0.0375 rpy=1.5708 0 0
- joint wheel3: origin xyz=-0.1055 0.10251 -0.0545 rpy=1.5708 0 0 -> xyz=-0.1055 0.1025 0.0375 rpy=1.5708 0 0
- joint wheel4: origin xyz=-0.1055 -0.1025 -0.0545 rpy=1.5708 0 0 -> xyz=-0.1055 -0.1025 0.0375 rpy=1.5708 0 0

Commit message: update

File: LGDXRobot2.urdf (robot description, URDF)
Before this commit: robot /Users/sam/Develop/lgdxrobot2-webots/LGDXRobot2.urdf, 26 links, 25 joints
Links:
- removed link solid_0
- removed link solid_1
- removed link solid_10
- removed link solid_2
- removed link solid_3
- removed link solid_4
- removed link solid_5
- removed link solid_6
- removed link solid_7
- removed link solid_8
- removed link solid_9
- added link BASE_CENTRE_SOLID; collision box size=0.124 0.237 0.004; visual box size=0.124 0.237 0.004
- added link BASE_FRONT_SOLID; collision box size=0.08 0.145 0.004; visual box size=0.08 0.145 0.004
- added link BASE_REAR_SOLID; collision box size=0.08 0.145 0.004; visual box size=0.08 0.145 0.004
- added link BASE_TOP_SOLID; collision box size=0.286 0.237 0.004; visual box size=0.286 0.237 0.004
Joints:
- removed joint base_link_solid_0_joint
- removed joint base_link_solid_1_joint
- removed joint base_link_solid_2_joint
- removed joint base_link_solid_3_joint
- removed joint base_link_solid_4_joint
- removed joint base_link_solid_5_joint
- removed joint base_link_solid_6_joint
- removed joint base_link_solid_7_joint
- removed joint base_link_solid_8_joint
- removed joint base_link_solid_9_joint
- removed joint base_link_solid_joint
- added joint base_link_BASE_CENTRE_SOLID_joint: type fixed, parent base_link, child BASE_CENTRE_SOLID, origin xyz=0 0 0.057 rpy=0 0 0
- added joint base_link_BASE_FRONT_SOLID_joint: type fixed, parent base_link, child BASE_FRONT_SOLID, origin xyz=0.102 0 0.057 rpy=0 0 0
- added joint base_link_BASE_REAR_SOLID_joint: type fixed, parent base_link, child BASE_REAR_SOLID, origin xyz=-0.102 0 0.057 rpy=0 0 0
- added joint base_link_BASE_TOP_SOLID_joint: type fixed, parent base_link, child BASE_TOP_SOLID, origin xyz=0 0 0.129 rpy=0 0 0
- joint lidar_secondary_motor: child solid_10 -> solid
